File: C128DKEYBOARD_ALT/C128DKEYBOARD.kicad_pcb (KiCad board)
At the start: 2 copper layers, 355.7 x 127.8 mm, 99 parts, among them J1 DB25_Male, K10 LINEFEED, K100 SPACE, K101 SHIFTLOCK, K102 DEAD, K103 CRSRUPDOWN, K104 CRSRLEFTRIGHT, K11 4080, K12 NOSCROLL, K13 POUND, K14 DEAD, K15 DEAD, K16 DEAD, K21 CLRHOME, K22 TAB, K23 UPARROW, K24 BACKARROW, K25 1, K26 2, K27 3, K28 4, K29 5, K30 6, K31 7, K32 8, K33 9, K34 0, K35 +, K36 -, K37 INSDEL, K4 ESC, K42 =, K43 DEAD, K44 DEAD, K45 CONTROL, K46 Q, K47 W, K48 E, K49 R, K5 F1, K50 T, K51 Y, K52 U, K53 I, K54 O, K55 P, K56 AT, K57 ASTERISK, K58 RESTORE, K6 F3, K62 RUNSTOP, K63 A, K64 S, K65 D, K66 F, K67 G, K68 H, K69 J, K7 F5, K70 K, K71 L, K72 :, K73 ;, K74 RETURN, K79 KEYPAD_UP, K8 F7, K80 SHIFTL, K81 Z, K82 X, K83 C, K84 V, K85 B, K86 N, K87 M, K88 ,, K89 ., K9 HELP, K90 /, K91 RSHIFT, K94 KEYPAD_LEFT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

Commit message: update layout
Parts:
- moved J1 7.87 mm to (353.8, 135.1)
- moved K21 1.68 mm to (356.8, 161.7)
- moved K22 1.68 mm to (375.8, 161.7)
- moved K23 1.68 mm to (394.9, 161.7)
- moved K42 1.68 mm to (356.8, 180.7)
- moved K43 1.68 mm to (375.8, 180.7)
- moved K44 1.68 mm to (394.9, 180.7)
- moved K79 1.68 mm to (375.8, 218.8)
- moved K94 1.68 mm to (356.8, 237.9)
- moved K95 1.68 mm to (375.8, 237.9)
- moved K96 1.68 mm to (394.9, 237.9)
Routing:
- net PIN23: track 480.1 -> 558.5 mm, vias 1 -> 0
- net PIN12: track 518.8 -> 593.0 mm, vias 3 -> 0
- net PIN7: track 513.8 -> 566.2 mm, vias 4 -> 1
- net PIN10: track 434.2 -> 484.5 mm, vias 0 -> 1
- net VCC: track 653.5 -> 609.6 mm
- net PIN6: track 507.2 -> 546.7 mm
- net PIN3: track 84.7 -> 53.2 mm, vias 1 -> 0
- net 4080LED: track 192.8 -> 162.4 mm, vias 1 -> 0
- net PIN18: track 357.7 -> 331.9 mm, vias 0 -> 2
- net PIN11: track 406.7 -> 382.7 mm, vias 1 -> 2
- net 4080TOGGLE: track 194.9 -> 176.4 mm, vias 1 -> 0
- net PIN5: track 442.1 -> 456.5 mm, vias 3 -> 1
- net PIN16: track 259.9 -> 245.6 mm, vias 0 -> 1
- net Net-(D4-A): track 26.6 -> 36.4 mm, vias 1 -> 0
- net PIN19: track 466.0 -> 456.5 mm, vias 2 -> 3
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Other:
- board size 355.7 x 127.8 mm -> 352 x 127.8 mm
